File: tiny2-41.kicad_pcb (KiCad board)
At the start: 2 copper layers, 10 parts, among them J1 Conn_02x07_Odd_Even, J2 Conn_01x04_Female, J3 Conn_01x08_Male, U1 4050, U2 CD40109BE, U3 Pico

Commit message: Updated
Parts:
- added J10: Conn_01x01_Male, TestPoint:TestPoint_Pad_1.0x1.0mm, F.Cu at (130.5, 149.9)
- added J11: Conn_01x01_Male, TestPoint:TestPoint_Pad_1.0x1.0mm, F.Cu at (132.3, 149.9)
- added J12: Conn_01x01_Male, TestPoint:TestPoint_Pad_1.0x1.0mm, F.Cu at (134.1, 149.9)
- added J2: Conn_01x01_Male, TestPoint:TestPoint_Pad_1.0x1.0mm, F.Cu at (115.9, 149.9)
- added J3: Conn_01x01_Male, TestPoint:TestPoint_Pad_1.0x1.0mm, F.Cu at (117.7, 149.9)
- added J4: Conn_01x01_Male, TestPoint:TestPoint_Pad_1.0x1.0mm, F.Cu at (119.6, 149.9)
- added J5: Conn_01x01_Male, TestPoint:TestPoint_Pad_1.0x1.0mm, F.Cu at (121.4, 149.9)
- added J6: Conn_01x01_Male, TestPoint:TestPoint_Pad_1.0x1.0mm, F.Cu at (123.2, 149.9)
- added J7: Conn_01x01_Male, TestPoint:TestPoint_Pad_1.0x1.0mm, F.Cu at (125.0, 149.9)
- added J8: Conn_01x01_Male, TestPoint:TestPoint_Pad_1.0x1.0mm, F.Cu at (126.8, 149.9)
- added J9: Conn_01x01_Male, TestPoint:TestPoint_Pad_1.0x1.0mm, F.Cu at (128.6, 149.9)
- J1: value Conn_02x07_Odd_Even -> Conn_01x01_Male; footprint Connector_IDC:IDC-Header_2x07_P2.54mm_Horizontal -> TestPoint:TestPoint_Pad_1.0x1.0mm
- moved J1 19.1 mm to (114.1, 149.9), turned to 0 degrees
- renumbered J2 to J20, J3 to J21

Commit message: Updated ...
Parts:
- added IC1: MB85RC1MTPNF-G-JNERE1, KiCad:SOIC127P600X175-8N, F.Cu at (138.4, 126.9)
- added RN1: R_Network06, KiCad:4607X101105LF, F.Cu at (114.7, 127.9)
- R2, R3: value 100k -> R
- moved U1 15.7 mm to (132.4, 137.1), turned to 180 degrees
- moved R2 13.0 mm to (139.7, 109.7)
- moved U2 11.5 mm to (120.4, 137.0), turned to 180 degrees
- moved D1 3.18 mm to (139.7, 72.4), turned to -90 degrees
- moved J10 2.64 mm to (132.9, 148.9)
- moved J8 2.64 mm to (129.3, 148.9)
- moved J1 2.64 mm to (116.6, 148.9)
- moved J4 2.64 mm to (122.0, 148.9)
- moved J5 2.64 mm to (123.8, 148.9)
- moved J6 2.64 mm to (125.6, 148.9)
- moved J7 2.64 mm to (127.5, 148.9)
- moved J11 2.64 mm to (134.7, 148.9)
- moved J12 2.64 mm to (136.6, 148.9)
- moved J2 2.64 mm to (118.4, 148.9)
- moved J3 2.64 mm to (120.2, 148.9)
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Connections:
- R2 pad 1: /DATA -> /+3.3V
- R2 pad 2: GND -> /SDA
- R3 pad 1: /ISA -> /+3.3V
- R3 pad 2: GND -> /SCL
- U3 pad 9: unconnected-(U3-Pad9) -> /FRAM_EN
